Commit message: [*] 缓存

File: cartographer_ros/urdf/backpack_2d.urdf (robot description, URDF)
Before this commit: robot cartographer_backpack_2d, 4 links, 3 joints
Links:
- removed link horizontal_laser_link
- removed link imu_link
- removed link vertical_laser_link
- added link odom; visual box size=0.06 0.04 0.02
- added link scan; visual cylinder length=0.05 radius=0.03
- link base_link: geometry visual box size=0.60 0.52 0.4
Joints:
- removed joint horizontal_laser_link_joint
- removed joint imu_link_joint
- removed joint vertical_laser_link_joint
- added joint odom_link_joint: type fixed, parent base_link, child odom, origin xyz=0 0 0.05 rpy=0 3.1415926 0
- added joint scan_joint: type fixed, parent base_link, child scan, origin xyz=0 0 0.1 rpy=0 3.1415926 3.1415926

Commit message: [*] 能跑通，但是地图有问题

File: cartographer_ros/urdf/backpack_2d.urdf (robot description, URDF)
Before this commit: robot agv, 3 links, 2 joints
Links:
- removed link odom
- removed link scan
- added link imu_link; visual box size=0.06 0.04 0.02
- added link laser; visual cylinder length=0.05 radius=0.03
- added link vertical_laser_link; visual cylinder length=0.05 radius=0.03
- link base_link: geometry 
Joints:
- removed joint odom_link_joint
- removed joint scan_joint
- added joint imu_link_joint: type fixed, parent base_link, child imu_link, origin xyz=0 0 0
- added joint laser_joint: type fixed, parent base_link, child laser, origin xyz=0.1007 0 0.0558
- added joint vertical_laser_link_joint: type fixed, parent base_link, child vertical_laser_link, origin xyz=0.1007 0 0.1814 rpy=0 -1.570796 3.141593
